File: HW/HW.sch (KiCad schematic (older format))
At the start: 64 parts, among them J1 PZT, J2 Barrel_Jack, J3 PRG, J4 PRG, U1 AD9834, U10 REF02CP, U2 25MHz, U3 NE5532, U4 AD8009AR, U5 NE5532, U6 MCP3201, U7 STM32F042F6Px, U8 TXS0108EPW, U9 AZ1117-5.0, Y1 8MHz

Commit message: add: gerber
Parts:
- removed C8, C9: 12p, symbol Device:C
- removed Y1: 8MHz, symbol Device:Crystal
- added C22, C23: 4.7uF, Capacitor_SMD:C_0603_1608Metric_Pad1.08x0.95mm_HandSolder, symbol Device:C
- added U10: AZ1117-3.3, Package_TO_SOT_SMD:SOT-223-3_TabPin2, symbol Regulator_Linear:AZ1117-3.3
- C1, C10, C11, C12, C13, C14, C18, C19, C2, C20, C21, C3, C4, C5, C6, C7: footprint (none) -> Capacitor_SMD:C_0603_1608Metric_Pad1.08x0.95mm_HandSolder
- C15: renamed from C16; footprint (none) -> Capacitor_SMD:C_Elec_6.3x5.4
- C16: renamed from C17; footprint (none) -> Capacitor_SMD:C_Elec_6.3x5.4
- C17: renamed from C15; footprint (none) -> Capacitor_SMD:C_0603_1608Metric_Pad1.08x0.95mm_HandSolder
- C24: renamed from C22; footprint (none) -> Capacitor_SMD:C_0603_1608Metric_Pad1.08x0.95mm_HandSolder
- C25: renamed from C23; footprint (none) -> Capacitor_SMD:C_0603_1608Metric_Pad1.08x0.95mm_HandSolder
- C26: renamed from C24; footprint (none) -> Capacitor_SMD:C_0603_1608Metric_Pad1.08x0.95mm_HandSolder
- D1, D2: footprint Diode_SMD:D_MiniMELF -> Diode_SMD:D_SOD-123
- D3, D4, D5: footprint (none) -> LED_SMD:LED_0603_1608Metric_Pad1.05x0.95mm_HandSolder
- J1: footprint (none) -> Connector_Coaxial:SMA_Amphenol_132289_EdgeMount
- J2: footprint (none) -> Connector_BarrelJack:BarrelJack_Horizontal
- J3: value PRG -> UART; footprint (none) -> Connector_PinHeader_2.54mm:PinHeader_1x04_P2.54mm_Vertical
- J4: footprint (none) -> Connector_PinHeader_2.54mm:PinHeader_1x04_P2.54mm_Vertical
- JP1: footprint Jumper:SolderJumper-2_P1.3mm_Open_TrianglePad1.0x1.5mm -> Jumper:SolderJumper-2_P1.3mm_Open_RoundedPad1.0x1.5mm
- R1, R10, R11, R12, R13, R16, R17, R2, R3, R4, R5, R6, R7, R8, R9: footprint (none) -> Resistor_SMD:R_0603_1608Metric_Pad0.98x0.95mm_HandSolder
- R14, R15: footprint (none) -> Resistor_SMD:R_0805_2012Metric_Pad1.20x1.40mm_HandSolder
- R18: value 330 -> 820; footprint (none) -> Resistor_SMD:R_0603_1608Metric_Pad0.98x0.95mm_HandSolder
- U11: renamed from U10; footprint Package_DIP:DIP-8_W7.62mm -> Package_SO:SOIC-8_3.9x4.9mm_P1.27mm
- U3, U5, U6: footprint (none) -> Package_SO:SOIC-8_3.9x4.9mm_P1.27mm
- U9: footprint (none) -> Package_TO_SOT_SMD:SOT-223-3_TabPin2
Connections:
- net +3V3: now also C23.1, U10.2 (VO)
- net +5V: now also C22.1, U10.3 (VI)
- net CLK: now also U8.5 (A4); no longer U8.1 (A1)
- net CS_1: now also U8.3 (A2); no longer U8.4 (A3)
- net GND: now also U1.10 (PSELECT), U1.11 (RESET), U1.12 (SLEEP), U1.9 (FSELECT), C22.2, C23.2, U10.1 (GND)
- net MISO: now also U8.4 (A3); no longer U8.3 (A2)
- net at U1.8 (MCLK), U2.3 (CLK): now also U7.2 (PF0)
- net B2: now reaches U6.5 (~CS~/SHDN)
- net B2: now also U8.18 (B2); no longer U8.17 (B3)
- net B3: now reaches U6.6 (Dout)
- net B3: now also U8.17 (B3); no longer U8.18 (B2)
- net at U8.20 (B1): no longer U6.7 (CLK)
- net B4: now reaches U8.16 (B4)
- net B4: now also U6.7 (CLK)
Other:
- moved on the sheet: C1, C10, C11, C12, C13, C14, C15, C16, C17, C18, C19, C2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
